File: wheel_self_balance.kicad_pcb (KiCad board)
At the start: 2 copper layers, 37 x 32.5 mm, 32 parts, among them J1 USB_B_Micro, SW1 SW_SPDT, U1 STM32F103C8T6, U2 AMS1117-3.3, Y1 16MHz

Commit message: Update image for readme
Other:
- board text added: "|Ver 1.0 Designed |by Tran Minh Nhat"
Changed lines of the file:
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@@
     (property "ki_keywords" "quartz ceramic resonator oscillator")
     (attr smd)
-    (fp_text reference "Y1" (at 0 2.6 -180) (layer "F.SilkS")
+    (fp_text reference "Y1" (at 2.15 2.48 -180) (layer "F.SilkS")
         (effects (font (size 1 1) (thickness 0.15)))
     )
@@
     (property "ki_keywords" "L ferrite bead inductor filter")
     (attr smd)
-    (fp_text reference "FB1" (at 2.3875 0.2 -180) (layer "F.SilkS")
+    (fp_text reference "FB1" (at 2.9875 1.6 -180) (layer "F.SilkS")
         (effects (font (size 1 1) (thickness 0.15)))
     )
@@
     (property "ki_keywords" "mounting hole")
     (attr exclude_from_pos_files)
-    (fp_text reference "H3" (at 1.15 -3.1) (layer "F.SilkS")
+    (fp_text reference "H3" (at 1.15 -3.1) (layer "F.SilkS") hide
         (effects (font (size 1 1) (thickness 0.15)))
     )
@@
     (property "ki_keywords" "R resistor")
     (attr smd)
-    (fp_text reference "R4" (at 0 1.3125) (layer "F.SilkS")
+    (fp_text reference "R4" (at -3.8 0.0125) (layer "F.SilkS")
         (effects (font (size 1 1) (thickness 0.15)))
     )
@@
     (property "ki_keywords" "mounting hole")
     (attr exclude_from_pos_files)
-    (fp_text reference "H2" (at 1.6 3.35) (layer "F.SilkS")
+    (fp_text reference "H2" (at 1.6 3.35) (layer "F.SilkS") hide
         (effects (font (size 1 1) (thickness 0.15)))
     )
@@
     (property "ki_keywords" "connector USB micro")
     (attr smd)
-    (fp_text reference "J1" (at 5.8 2.4 180) (layer "F.SilkS")
+    (fp_text reference "J1" (at -0.2 0.4 180) (layer "F.SilkS")
         (effects (font (size 1 1) (thickness 0.15)))
     )
@@
     (property "ki_keywords" "capacitor cap")
     (attr smd)
-    (fp_text reference "C11" (at -1.8 -1.15 180) (layer "F.SilkS")
+    (fp_text reference "C11" (at -1.8 -1.03 180) (layer "F.SilkS")
         (effects (font (size 1 1) (thickness 0.15)))
     )
@@
     (property "ki_keywords" "R resistor")
     (attr smd)
-    (fp_text reference "R2" (at -1.7 0.1) (layer "F.SilkS")
+    (fp_text reference "R2" (at -1.2 1.4) (layer "F.SilkS")
         (effects (font (size 1 1) (thickness 0.15)))
     )
@@
     (property "ki_keywords" "mounting hole")
     (attr exclude_from_pos_files)
-    (fp_text reference "H4" (at 0 -3.2) (layer "F.SilkS")
+    (fp_text reference "H4" (at 0 -3.2) (layer "F.SilkS") hide
         (effects (font (size 1 1) (thickness 0.15)))
     )
@@
     (property "ki_keywords" "capacitor cap")
     (attr smd)
-    (fp_text reference "C4" (at 0.1 -1.4 180) (layer "F.SilkS")
+    (fp_text reference "C4" (at 0.75 1.45 180) (layer "F.SilkS")
         (effects (font (size 1 1) (thickness 0.15)))
     )
@@
     (property "ki_keywords" "LED diode")
     (attr smd)
-    (fp_text reference "D1" (at -2.2125 -1.5 -180) (layer "F.SilkS")
+    (fp_text reference "D1" (at -0.7625 -3.25 -180) (layer "F.SilkS")
         (effects (font (size 1 1) (thickness 0.15)))
     )
@@
     (property "ki_keywords" "capacitor cap")
     (attr smd)
-    (fp_text reference "C6" (at -1.7 -0.3) (layer "F.SilkS")
+    (fp_text reference "C6" (at -1.75 -1.2) (layer "F.SilkS")
         (effects (font (size 1 1) (thickness 0.15)))
     )
@@
     (property "ki_keywords" "mounting hole")
     (attr exclude_from_pos_files)
-    (fp_text reference "H1" (at 3.2 2.2) (layer "F.SilkS")
+    (fp_text reference "H1" (at 3.2 2.2) (layer "F.SilkS") hide
         (effects (font (size 1 1) (thickness 0.15)))
     )
@@
     (property "ki_keywords" "R resistor")
     (attr smd)
-    (fp_text reference "R3" (at -1.7 -0.3) (layer "F.SilkS")
+    (fp_text reference "R3" (at -1.55 -1.25) (layer "F.SilkS")
         (effects (font (size 1 1) (thickness 0.15)))
     )
@@
     (property "ki_keywords" "capacitor cap")
     (attr smd)
-    (fp_text reference "C1" (at -1.88 0.5) (layer "F.SilkS")
+    (fp_text reference "C1" (at -1.88 0.2) (layer "F.SilkS")
         (effects (font (size 1 1) (thickness 0.15)))
     )
@@
     (property "ki_keywords" "Arm Cortex-M3 STM32F1 STM32F103")
     (attr smd)
-    (fp_text reference "U1" (at 4.25 -4.6) (layer "F.SilkS")
+    (fp_text reference "U1" (at 0.15 -0.3) (layer "F.SilkS")
         (effects (font (size 1 1) (thickness 0.15)))
     )
@@
     (property "ki_keywords" "capacitor cap")
     (attr smd)
-    (fp_text reference "C10" (at 0.1 1.75 180) (layer "F.SilkS")
+    (fp_text reference "C10" (at 0.65 2.07 180) (layer "F.SilkS")
         (effects (font (size 1 1) (thickness 0.15)))
     )
@@
   (gr_arc (start 99 76.5) (mid 99.878679 74.378679) (end 102 73.5)
     (stroke (width 0.2) (type default)) (layer "Edge.Cuts"))
+  (gr_text "|Ver 1.0 Designed\n|by Tran Minh Nhat" (at 118.6 82.95) (layer "F.SilkS")
+    (effects (font (size 1 1) (thickness 0.15)) (justify left bottom))
+  )
   (segment (start 109.2 99.15) (end 110.45 100.4) (width 0.5) (layer "F.Cu") (net 1))
   (segment (start 118.5 104.15) (end 118.5 101.05) (width 0.5) (layer "F.Cu") (net 1))
